File: ergogen/output/pcbs/Blasphemy.kicad_pcb (KiCad board)
At the start: 2 copper layers, 255.1 x 95.5 mm, 46 parts

Commit message: update config
Parts:
- added D1: , ComboDiode, F.Cu at (-0.61, 4.96)
- added D10: , ComboDiode, F.Cu at (136.1, 15.1)
- added D11: , ComboDiode, F.Cu at (-0.57, 24.1)
- added D12: , ComboDiode, F.Cu at (20.6, 26.7)
- added D13: , ComboDiode, F.Cu at (39.5, 29.0)
- added D14: , ComboDiode, F.Cu at (58.4, 31.3)
- added D15: , ComboDiode, F.Cu at (81.9, 34.2)
- added D16: , ComboDiode, F.Cu at (218.5, 24.1)
- added D17: , ComboDiode, F.Cu at (197.3, 26.7)
- added D18: , ComboDiode, F.Cu at (178.4, 29.0)
- added D19: , ComboDiode, F.Cu at (159.6, 31.3)
- added D2: , ComboDiode, F.Cu at (18.2, 7.28)
- added D20: , ComboDiode, F.Cu at (136.0, 34.2)
- added D21: , ComboDiode, F.Cu at (-5.24, 42.7)
- added D22: , ComboDiode, F.Cu at (13.6, 45.0)
- added D23: , ComboDiode, F.Cu at (32.5, 47.3)
- added D24: , ComboDiode, F.Cu at (51.3, 49.6)
- added D25: , ComboDiode, F.Cu at (77.3, 52.8)
- added D26: , ComboDiode, F.Cu at (223.2, 42.7)
- added D27: , ComboDiode, F.Cu at (204.3, 45.0)
- added D28: , ComboDiode, F.Cu at (185.5, 47.3)
- added D29: , ComboDiode, F.Cu at (166.6, 49.6)
- added D3: , ComboDiode, F.Cu at (37.1, 9.59)
- added D30: , ComboDiode, F.Cu at (140.7, 52.8)
- added D31: , ComboDiode, F.Cu at (37.2, 67.0)
- added D32: , ComboDiode, F.Cu at (63.2, 70.2)
- added D33: , ComboDiode, F.Cu at (82.0, 72.5)
- added D34: , ComboDiode, F.Cu at (180.7, 67.0)
- added D35: , ComboDiode, F.Cu at (154.8, 70.2)
- added D36: , ComboDiode, F.Cu at (135.9, 72.5)
- added D4: , ComboDiode, F.Cu at (56.0, 11.9)
- added D5: , ComboDiode, F.Cu at (81.9, 15.1)
- added D6: , ComboDiode, F.Cu at (218.6, 4.96)
- added D7: , ComboDiode, F.Cu at (199.7, 7.28)
- added D8: , ComboDiode, F.Cu at (180.8, 9.59)
- added D9: , ComboDiode, F.Cu at (162.0, 11.9)
